File: KiCad/CrudeCameraSheild.kicad_pcb (KiCad board)
At the start: 2 copper layers, 93.5 x 53.5 mm, 284 parts, among them J1 GPIO, Q1 ALS-PT19, Q10 ALS-PT19, Q100 ALS-PT19, Q101 ALS-PT19, Q102 ALS-PT19, Q103 ALS-PT19, Q104 ALS-PT19, Q105 ALS-PT19, Q106 ALS-PT19, Q107 ALS-PT19, Q108 ALS-PT19, Q109 ALS-PT19, Q11 ALS-PT19, Q110 ALS-PT19, Q111 ALS-PT19, Q112 ALS-PT19, Q113 ALS-PT19, Q114 ALS-PT19, Q115 ALS-PT19, Q116 ALS-PT19, Q117 ALS-PT19, Q118 ALS-PT19, Q119 ALS-PT19, Q12 ALS-PT19, Q120 ALS-PT19, Q121 ALS-PT19, Q122 ALS-PT19, Q123 ALS-PT19, Q124 ALS-PT19, Q125 ALS-PT19, Q126 ALS-PT19, Q127 ALS-PT19, Q128 ALS-PT19, Q129 ALS-PT19, Q13 ALS-PT19, Q130 ALS-PT19, Q131 ALS-PT19, Q132 ALS-PT19, Q133 ALS-PT19, Q134 ALS-PT19, Q135 ALS-PT19, Q136 ALS-PT19, Q137 ALS-PT19, Q138 ALS-PT19, Q139 ALS-PT19, Q14 ALS-PT19, Q140 ALS-PT19, Q141 ALS-PT19, Q142 ALS-PT19, Q143 ALS-PT19, Q144 ALS-PT19, Q145 ALS-PT19, Q146 ALS-PT19, Q147 ALS-PT19, Q148 ALS-PT19, Q149 ALS-PT19, Q15 ALS-PT19, Q150 ALS-PT19, Q151 ALS-PT19, Q152 ALS-PT19, Q153 ALS-PT19, Q154 ALS-PT19, Q155 ALS-PT19, Q156 ALS-PT19, Q157 ALS-PT19, Q158 ALS-PT19, Q159 ALS-PT19, Q16 ALS-PT19, Q160 ALS-PT19, Q161 ALS-PT19, Q162 ALS-PT19, Q163 ALS-PT19, Q164 ALS-PT19, Q165 ALS-PT19, Q166 ALS-PT19, Q167 ALS-PT19, Q168 ALS-PT19, Q169 ALS-PT19, Q17 ALS-PT19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

Commit message: Corrected spelling of sensor on silkscreen. Updated resistor values.
Other:
- board text added: "Crude Camera Sensor V1.1"
- board text removed: "Crude Camera Senor V1.0"
Changed lines of the file:
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@@
-(kicad_pcb (version 20171130) (host pcbnew "(5.1.4)-1")
+(kicad_pcb (version 20171130) (host pcbnew "(5.1.5)-3")
   (general
     (thickness 1.6)
@@
   )
   (page A4)
+  (title_block
+    (title "Crude Camera Sensor")
+    (date 2020-02-04)
+    (rev 1.1)
+    (company "Northeastern Wireless Club")
+  )
   (layers
     (0 F.Cu signal)
@@
     (add_net "Net-(J1-Pad8)")
     (add_net "Net-(J1-Pad9)")
-    (add_net "Net-(SHIELD1-Pad0)")
-    (add_net "Net-(SHIELD1-Pad1)")
-    (add_net "Net-(SHIELD1-Pad10)")
-    (add_net "Net-(SHIELD1-Pad11)")
-    (add_net "Net-(SHIELD1-Pad12)")
-    (add_net "Net-(SHIELD1-Pad13)")
-    (add_net "Net-(SHIELD1-Pad14)")
-    (add_net "Net-(SHIELD1-Pad15)")
-    (add_net "Net-(SHIELD1-Pad16)")
-    (add_net "Net-(SHIELD1-Pad17)")
-    (add_net "Net-(SHIELD1-Pad18)")
-    (add_net "Net-(SHIELD1-Pad19)")
     (add_net "Net-(SHIELD1-Pad2)")
     (add_net "Net-(SHIELD1-Pad3)")
-    (add_net "Net-(SHIELD1-Pad38)")
-    (add_net "Net-(SHIELD1-Pad39)")
-    (add_net "Net-(SHIELD1-Pad3V3)")
-    (add_net "Net-(SHIELD1-Pad4)")
-    (add_net "Net-(SHIELD1-Pad40)")
-    (add_net "Net-(SHIELD1-Pad41)")
-    (add_net "Net-(SHIELD1-Pad5)")
-    (add_net "Net-(SHIELD1-Pad50)")
-    (add_net "Net-(SHIELD1-Pad51)")
-    (add_net "Net-(SHIELD1-Pad52)")
-    (add_net "Net-(SHIELD1-Pad53)")
-    (add_net "Net-(SHIELD1-Pad5V)")
-    (add_net "Net-(SHIELD1-Pad6)")
-    (add_net "Net-(SHIELD1-Pad7)")
-    (add_net "Net-(SHIELD1-Pad8)")
-    (add_net "Net-(SHIELD1-Pad9)")
-    (add_net "Net-(SHIELD1-PadAREF)")
-    (add_net "Net-(SHIELD1-PadV_IN)")
   )
   (net_class Power ""
@@
     (pad 14 thru_hole oval (at 68.58 -50.8 90) (size 2.54 1.524) (drill 0.8128) (layers *.Cu *.Mask F.SilkS))
   )
-  (gr_text "Crude Camera Senor V1.0" (at 178.5 78.5 90) (layer F.SilkS)
+  (gr_text "Crude Camera Sensor V1.1" (at 178.5 78.5 90) (layer F.SilkS)
     (effects (font (size 1 1) (thickness 0.15)))
   )
